Commit message: feat lander model

File: scripts/lander.urdf (robot description, URDF)
Before this commit: robot lunar_lander, 5 links, 4 joints
Links:
- removed link base
- removed link leg_1
- removed link leg_2
- removed link thruster_left
- removed link thruster_right
- added link base_link, mass 10.0; collision box size=1.0 1.0 1.3; visual box size=1.0 1.0 1.3
- added link leg1_link, mass 1.0; collision box size=0.3 0.3 0.8; visual box size=0.3 0.3 0.8
- added link leg2_link, mass 1.0; collision box size=0.3 0.3 0.8; visual box size=0.3 0.3 0.8
- added link leg3_link, mass 1.0; collision box size=0.3 0.3 0.8; visual box size=0.3 0.3 0.8
- added link leg4_link, mass 1.0; collision box size=0.3 0.3 0.8; visual box size=0.3 0.3 0.8
Joints:
- removed joint leg_1_joint
- removed joint leg_2_joint
- removed joint thruster_left_joint
- removed joint thruster_right_joint
- added joint leg1_PrismaticJoint: type prismatic, parent base_link, child leg1_link, origin xyz=-0.2432818 0.2807126 -1.7951556 rpy=0.0094365 -0.0100893 0.0664074, axis 0. 0. 1., limit lower=0.0 upper=0.2 effort=100.0 velocity=1.0
- added joint leg2_PrismaticJoint: type prismatic, parent base_link, child leg2_link, origin xyz=-0.2313453 1.682129 -1.3760384 rpy=0.56972 0.0418672 -0.0910576, axis 0. 0. 1., limit lower=0.0 upper=0.2 effort=100.0 velocity=1.0
- added joint leg3_PrismaticJoint: type prismatic, parent base_link, child leg3_link, origin xyz=-1.4118276 0.1897153 -1.4576046 rpy=0.0056381 0.5710402 0.0709048, axis 0. 0. 1., limit lower=0.0 upper=0.2 effort=100.0 velocity=1.0
- added joint leg4_PrismaticJoint: type prismatic, parent base_link, child leg4_link, origin xyz=-1.399891 1.5911317 -1.0384876 rpy=0.6647065 0.5208261 0.2558816, axis 0. 0. 1., limit lower=0.0 upper=0.2 effort=100.0 velocity=1.0
